File: Hardware/Rele Wifi/relay-wifi-kc.kicad_sch (KiCad schematic)
At the start: 47 parts, among them J1 SalidaRele1, J2 SalidaRele2, J3 SalidaRele3, J4 SalidaRele4, K1 RELAY_C, K2 RELAY_C, K3 RELAY_C, K4 RELAY_C, Q1 TO23, Q2 TO23, Q3 TO23, Q4 TO23, U1 LM78M05_TO220, U2 ESP32_DevKit_V1_DOIT, U3 PC817, U4 PC817, U5 PC817, U6 PC817

Commit message: Esquematico y PCB V3
Parts:
- D10, D12, D2, D3, D4, D5, D6, D8: footprint Diode_SMD:D_0805_2012Metric_Pad1.15x1.40mm_HandSolder -> Diode_SMD:D_SMA
Connections:
- net 5V: now also U3.4, U4.4, U5.4, U6.4
- net at R9.2: now also D13.2 (A); no longer D13.1 (K)
- net at Q4.2 (B), R5.1: no longer D13.2 (A)
- net at R6.2: now also D7.2 (A); no longer D7.1 (K)
- net at R3.2: now also U4.3; no longer U4.4
- net at R7.2: now also D11.2 (A); no longer D11.1 (K)
- net at Q2.2 (B), R4.1: no longer D11.2 (A)
- net at R8.2: now also D9.2 (A); no longer D9.1 (K)
- net at Q3.2 (B), R3.1: no longer D9.2 (A)
- net at Q1.2 (B), R2.1: no longer D7.2 (A)
- net at R2.2: now also U3.3; no longer U3.4
- net at R4.2: now also U5.3; no longer U5.4
- net at R5.2: now also U6.3; no longer U6.4
- removed net GND+: C1.2, C2.2, D1.1 (K), D2.2 (A), D5.2 (A), Q1.3 (E), Q2.3 (E), Q3.3 (E), Q4.3 (E), R6.1, R7.1, R8.1, R9.1, U1.2 (GND), U3.3, U4.3, U5.3, U6.3
- net GND- renamed GND
- net GND: now also C1.2, C2.2, D1.1 (K), D11.1 (K), D13.1 (K), D2.2 (A), D5.2 (A), D7.1 (K), D9.1 (K), U1.2 (GND)
- new net: Q4.3 (E), R9.1
- new net: Q1.3 (E), R6.1
- new net: Q3.3 (E), R8.1
- new net: Q2.3 (E), R7.1
Other:
- moved on the sheet: D11, D13, D7, D9, J1, R10, R11, R12, R13, R6, R7, R8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
